File: pcb/DonConIOmini/DonConIOmini.kicad_sch (KiCad schematic)
At the start: 93 parts, among them J1 Ka Left, J2 Don Left, J3 Don Right, J4 Ka Right, J5 Pad, U1 TL074, U2 TL074, U3 RP2040-Zero, U5 MCP3204, U6 MCP1541-TT, U7 TXB0104D

Commit message: Update DonConIOmini PCB to rev 2.1
Add SERVICE, COIN, and TEST signal connections on previously
unconnected GP0-GP2 pins. Add 1x04 connectors for the new signals.

Co-Authored-By: Claude Opus 4.6 <noreply@anthropic.com>
Parts:
- added J6: SERVICE, Connector_JST:JST_XH_S4B-XH-A_1x04_P2.50mm_Horizontal, symbol Connector:Conn_01x04_Pin
Connections:
- net GND: now also J6.1 (Pin_1)
- net COIN: now reaches U3.10 (GP0)
- net COIN: now also J6.4 (Pin_4)
- net TEST: now reaches U3.11 (GP1)
- net TEST: now also J6.3 (Pin_3)
- net SERVICE: now reaches U3.12 (GP2)
- net SERVICE: now also J6.2 (Pin_2)
- no-connect marks 13 -> 10
Other:
- moved on the sheet: H1, H2, H3, H4, U3
